File: motor_pcb/motor-board-project.kicad_pcb (KiCad board)
At the start: 2 copper layers, 56 x 55.3 mm, 19 parts, among them J1 MOTOR_A, J2 MOTOR_B, J3 Conn_01x06, J4 12V_IN, U1 H450_module, U2 LM78L05_TO92

Commit message: Add files via upload
Parts:
- moved H4 31.6 mm to (118.3, 73.4)
- moved H3 4.96 mm to (118.3, 101.3)
- moved H2 2.92 mm to (67.5, 58.2)
Changed lines of the file:
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@@
   )
   (footprint "User Global Library:HOLE_BARE_3.1mm" (layer "F.Cu")
-    (at 70 59.7)
+    (at 67.5 58.2)
     (property "Sheetfile" "motor-board-project.kicad_sch")
     (property "Sheetname" "")
@@
   )
   (footprint "User Global Library:HOLE_BARE_3.1mm" (layer "F.Cu")
-    (at 115 105)
+    (at 118.3 101.3)
     (property "Sheetfile" "motor-board-project.kicad_sch")
     (property "Sheetname" "")
@@
   )
   (footprint "User Global Library:HOLE_BARE_3.1mm" (layer "F.Cu")
-    (at 120 105)
-    (property "Sheetfile" "motor-board-project.kicad_sch")
-    (property "Sheetname" "")
+    (at 118.3 73.4)
+    (property "Sheetfile" "motor-board-project.kicad_sch")
+    (property "Sheetname" "")
